File: PicoVersion/HW/13cmPico/rAD8348_Receiver/rAD8348_Receiver.kicad_sch (KiCad schematic)
At the start: 60 parts

Commit message: receiver mods
Parts:
- added C1, C2, C3, C4: 0u1, Capacitor_SMD:C_0805_2012Metric, symbol Device:C
- added R1, R3, R4: 200, Resistor_SMD:R_0805_2012Metric, symbol Device:R
- added R2: 3K9, Resistor_SMD:R_0805_2012Metric, symbol Device:R
- added R5, R6: 1K, Resistor_SMD:R_0805_2012Metric, symbol Device:R
- added R7: 10, Resistor_SMD:R_0805_2012Metric, symbol Device:R
- added RV1, RV2, RV3: 5K, symbol Device:R_Potentiometer_Small
- added U1: ADA4898-2, Package_SO:SOIC-8-1EP_3.9x4.9mm_P1.27mm_EP2.41x3.81mm, symbol Amplifier_Operational:ADA4898-2
- C101, C103, C107, C109, C111, C115, C119, C122, C123, C124: renamed from U; value (none) -> 1000p; footprint (none) -> Capacitor_SMD:C_0805_2012Metric
- C102, C104, C108, C110, C112: renamed from U; value (none) -> 0.01u; footprint (none) -> Capacitor_SMD:C_0805_2012Metric
- C105: renamed from U; value (none) -> 22u; footprint (none) -> Enevo:0603_CAP
- C106: renamed from U; value (none) -> 1500u; footprint (none) -> Capacitor_SMD:CP_Elec_10x10
- C113, C114: renamed from U; value (none) -> 0.01uF; footprint (none) -> Capacitor_SMD:C_0805_2012Metric
- C116: renamed from U; value (none) -> 10u; footprint (none) -> Capacitor_SMD:C_1206_3216Metric
- C117: renamed from U; value (none) -> 470p; footprint (none) -> Capacitor_SMD:C_0805_2012Metric
- C118: renamed from U; value (none) -> 0.0015uF; footprint (none) -> Capacitor_SMD:C_0805_2012Metric
- C120, C121: renamed from U; value (none) -> 4p3; footprint (none) -> Capacitor_SMD:C_0805_2012Metric
- C125, C131: renamed from U; value (none) -> 150p; footprint (none) -> Capacitor_SMD:C_0805_2012Metric
- C126, C129: renamed from U; value (none) -> 82p; footprint (none) -> Capacitor_SMD:C_0805_2012Metric
- C127, C128: renamed from U; value (none) -> 8p2; footprint (none) -> Capacitor_SMD:C_0805_2012Metric
- C130, C132: renamed from U; value (none) -> 4p7; footprint (none) -> Capacitor_SMD:C_0805_2012Metric
- C133: renamed from U; value (none) -> 0u1; footprint (none) -> Capacitor_SMD:C_0805_2012Metric
- L101, L102: renamed from U; value (none) -> 100n; footprint (none) -> Inductor_SMD:L_0805_2012Metric
- L103, L104: renamed from U; value (none) -> 8n7; footprint (none) -> Inductor_SMD:L_0805_2012Metric
- L105, L108: renamed from U; value (none) -> 1.2uH; footprint (none) -> Inductor_SMD:L_0805_2012Metric
- L106, L107: renamed from U; value (none) -> 0.68uH; footprint (none) -> Inductor_SMD:L_0805_2012Metric
- R101: renamed from U; value (none) -> 57.6; footprint (none) -> Resistor_SMD:R_0805_2012Metric
- R102: renamed from U; value (none) -> 174; footprint (none) -> Resistor_SMD:R_0805_2012Metric
- R103, R109: renamed from U; value (none) -> 200; footprint (none) -> Resistor_SMD:R_0805_2012Metric
- R104: renamed from U; value (none) -> 50; footprint (none) -> Resistor_SMD:R_0805_2012Metric
- R105, R107: renamed from U; value (none) -> 2K; footprint (none) -> Resistor_SMD:R_0805_2012Metric
- R106: renamed from U; value (none) -> 4K7; footprint (none) -> Resistor_SMD:R_0805_2012Metric
- R108, R112: renamed from U; value (none) -> 100; footprint (none) -> Resistor_SMD:R_0805_2012Metric
- R110, R111, R113, R114: renamed from U; value (none) -> 2; footprint (none) -> Resistor_SMD:R_0805_2012Metric
- R115, R116: renamed from U; value (none) -> 3K9; footprint (none) -> Resistor_SMD:R_0805_2012Metric
- U101: renamed from U; Description_1 (none) -> 50 MHz to 1000 MHz Quadrature Demodulator
- U102: renamed from U; value ADF4360-5BCP -> ADF4360-4; footprint ADF4360-5BCP:QFN50P400X400X100-25N -> adf4360:QFN50P400X400X100-25N
- renumbered U to U103
Connections:
- net GND: now also C1.2, C2.2, C3.2, C4.2, R1.2, R3.2, R4.2, R6.2, U1.4 (V-), U1.5 (+)
- net VCMO: now reaches C125.1, C126.2, C129.1, C131.1, R108.1, R112.2, U101.5 (VCMO)
- net VCMO: now also R7.2, U1.2 (-)
- net DEM_5V: now reaches C101.2, C102.2, C103.2, C104.2, R115.2, R116.2, U101.12 (VPS2), U101.2 (VPOS1), U101.20 (VPOS3)
- net DEM_5V: now also R2.1, R5.1, RV2.1, RV2.2, RV3.1, RV3.2, U1.8 (V+)
- net IOFS: now reaches U101.13 (IOFS)
- net IOFS: now also C3.1, R4.1, RV3.3
- net QOFS: now reaches U101.16 (QOFS)
- net QOFS: now also C2.1, R3.1, RV2.3
- net at U101.17 (VGIN): now also RV1.2
- new net: R7.1, U1.1
- new net: C4.1, R5.2, R6.1, U1.3 (+)
- new net: C1.1, R1.1, RV1.3
- new net: R2.2, RV1.1
- new net: U1.6 (-), U1.7
- no-connect marks 4 -> 2
Other:
- note added: "AD8348 IQ DEMODULATOR"
- note added: "TCXO REFIN UYNUTMA"
- moved on the sheet: C101, C102, C103, C104, C122, C123, C124, C125, C126, C127, C128, C129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
